File: proto.kicad_sch (KiCad schematic)
At the start: 12 parts, among them J1 Conn_01x05, J5 Conn_01x04, J6 Conn_01x05, J7 Conn_01x05, J8 Conn_01x03

Commit message: Populate Board
Parts:
- renumbered C23 to C?, C22 to C?, C28 to C?, F2 to F?, J1 to J?, J6 to J?, J5 to J?, J7 to J?, J8 to J?, R63 to R?, R62 to R?, R54 to R?
Changed lines of the file:
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@@
 		(on_board yes)
 		(dnp no)
-		(property "Reference" "J1"
+		(property "Reference" "J?"
 			(at 104.902 94.1832 0)
 			(effects
@@
 			(project "v0.4.4d"
 				(path "/5a477c6c-8a44-40c8-a075-f8fcd765b0eb/00000000-0000-0000-0000-00005cdc3535"
-					(reference "J1")
+					(reference "J?")
 					(unit 1)
 				)
@@
 		(on_board yes)
 		(dnp no)
-		(property "Reference" "J6"
+		(property "Reference" "J?"
 			(at 129.032 94.1832 0)
 			(effects
@@
 			(project "v0.4.4d"
 				(path "/5a477c6c-8a44-40c8-a075-f8fcd765b0eb/00000000-0000-0000-0000-00005cdc3535"
-					(reference "J6")
+					(reference "J?")
 					(unit 1)
 				)
@@
 		(on_board yes)
 		(dnp no)
-		(property "Reference" "#PWR072"
+		(property "Reference" "#PWR?"
 			(at 119.38 82.55 0)
 			(effects
@@
 			(project "v0.4.4d"
 				(path "/5a477c6c-8a44-40c8-a075-f8fcd765b0eb/00000000-0000-0000-0000-00005cdc3535"
-					(reference "#PWR072")
+					(reference "#PWR?")
 					(unit 1)
 				)
@@
 		(on_board yes)
 		(dnp no)
-		(property "Reference" "J5"
+		(property "Reference" "J?"
 			(at 156.0068 103.632 0)
 			(effects
@@
 			(project "v0.4.4d"
 				(path "/5a477c6c-8a44-40c8-a075-f8fcd765b0eb/00000000-0000-0000-0000-00005cdc3535"
-					(reference "J5")
+					(reference "J?")
 					(unit 1)
 				)
@@
 		(on_board yes)
 		(dnp no)
-		(property "Reference" "R63"
+		(property "Reference" "R?"
 			(at 153.4922 77.47 90)
 			(effects
@@
 				)
 				(path "/5a477c6c-8a44-40c8-a075-f8fcd765b0eb/00000000-0000-0000-0000-00005cdc3535"
-					(reference "R63")
+					(reference "R?")
 					(unit 1)
 				)
@@
 		(on_board yes)
 		(dnp no)
-		(property "Reference" "C23"
+		(property "Reference" "C?"
 			(at 166.4716 63.119 0)
 			(effects
@@
 				)
 				(path "/5a477c6c-8a44-40c8-a075-f8fcd765b0eb/00000000-0000-0000-0000-00005cdc3535"
-					(reference "C23")
+					(reference "C?")
 					(unit 1)
 				)
@@
 		(on_board yes)
 		(dnp no)
-		(property "Reference" "R62"
+		(property "Reference" "R?"
 			(at 161.4678 77.47 90)
 			(effects
@@
 				)
 				(path "/5a477c6c-8a44-40c8-a075-f8fcd765b0eb/00000000-0000-0000-0000-00005cdc3535"
-					(reference "R62")
+					(reference "R?")
 					(unit 1)
 				)
@@
 		(on_board yes)
 		(dnp no)
-		(property "Reference" "C22"
+		(property "Reference" "C?"
 			(at 148.4884 68.961 0)
 			(effects
@@
 				)
 				(path "/5a477c6c-8a44-40c8-a075-f8fcd765b0eb/00000000-0000-0000-0000-00005cdc3535"
-					(reference "C22")
+					(reference "C?")
 					(unit 1)
 				)
@@
 		(on_board yes)
 		(dnp no)
-		(property "Reference" "#PWR073"
+		(property "Reference" "#PWR?"
 			(at 133.35 66.04 0)
 			(effects
@@
 			(project "v0.4.4d"
 				(path "/5a477c6c-8a44-40c8-a075-f8fcd765b0eb/00000000-0000-0000-0000-00005cdc3535"
-					(reference "#PWR073")
+					(reference "#PWR?")
 					(unit 1)
 				)
@@
 		(on_board yes)
 		(dnp no)
-		(property "Reference" "#PWR074"
+		(property "Reference" "#PWR?"
 			(at 181.61 66.04 0)
 			(effects
@@
 			(project "v0.4.4d"
 				(path "/5a477c6c-8a44-40c8-a075-f8fcd765b0eb/00000000-0000-0000-0000-00005cdc3535"
-					(reference "#PWR074")
+					(reference "#PWR?")
 					(unit 1)
 				)
@@
 		(on_board yes)
 		(dnp no)
-		(property "Reference" "J7"
+		(property "Reference" "J?"
 			(at 104.902 111.9632 0)
 			(effects
@@
 			(project "v0.4.4d"
 				(path "/5a477c6c-8a44-40c8-a075-f8fcd765b0eb/00000000-0000-0000-0000-00005cdc3535"
-					(reference "J7")
+					(reference "J?")
 					(unit 1)
 				)
@@
 		(on_board yes)
 		(dnp no)
-		(property "Reference" "J8"
+		(property "Reference" "J?"
 			(at 135.382 111.9632 0)
 			(effects
@@
 			(project "v0.4.4d"
 				(path "/5a477c6c-8a44-40c8-a075-f8fcd765b0eb/00000000-0000-0000-0000-00005cdc3535"
-					(reference "J8")
+					(reference "J?")
 					(unit 1)
 				)
@@
 		(on_board yes)
 		(dnp no)
-		(property "Reference" "F2"
+		(property "Reference" "F?"
 			(at 96.2152 78.8416 0)
 			(effects
@@
 			(project "v0.4.4d"
 				(path "/5a477c6c-8a44-40c8-a075-f8fcd765b0eb/00000000-0000-0000-0000-00005cdc3535"
-					(reference "F2")
+					(reference "F?")
 					(unit 1)
 				)
@@
 		(on_board yes)
 		(dnp no)
-		(property "Reference" "#PWR0120"
+		(property "Reference" "#PWR?"
 			(at 93.98 80.01 0)
 			(effects
@@
 			(project "v0.4.4d"
 				(path "/5a477c6c-8a44-40c8-a075-f8fcd765b0eb/00000000-0000-0000-0000-00005cdc3535"
-					(reference "#PWR0120")
+					(reference "#PWR?")
 					(unit 1)
 				)
@@
 		(on_board yes)
 		(dnp no)
-		(property "Reference" "R54"
+		(property "Reference" "R?"
 			(at 204.6478 96.52 90)
 			(effects
@@
 				)
 				(path "/5a477c6c-8a44-40c8-a075-f8fcd765b0eb/00000000-0000-0000-0000-00005cdc3535"
-					(reference "R54")
+					(reference "R?")
 					(unit 1)
 				)
@@
 		(on_board yes)
 		(dnp no)
-		(property "Reference" "C28"
+		(property "Reference" "C?"
 			(at 211.201 95.3516 0)
 			(effects
@@
 				)
 				(path "/5a477c6c-8a44-40c8-a075-f8fcd765b0eb/00000000-0000-0000-0000-00005cdc3535"
-					(reference "C28")
+					(reference "C?")
 					(unit 1)
 				)
@@
 		(on_board yes)
 		(dnp no)
-		(property "Reference" "#PWR0121"
+		(property "Reference" "#PWR?"
 			(at 208.28 86.36 0)
 			(effects
@@
 			(project "v0.4.4d"
 				(path "/5a477c6c-8a44-40c8-a075-f8fcd765b0eb/00000000-0000-0000-0000-00005cdc3535"
-					(reference "#PWR0121")
+					(reference "#PWR?")
 					(unit 1)
 				)
@@
 		(on_board yes)
 		(dnp no)
-		(property "Reference" "#PWR0122"
+		(property "Reference" "#PWR?"
 			(at 199.39 96.52 0)
 			(effects
@@
 			(project "v0.4.4d"
 				(path "/5a477c6c-8a44-40c8-a075-f8fcd765b0eb/00000000-0000-0000-0000-00005cdc3535"
-					(reference "#PWR0122")
-					(unit 1)
-				)
+					(reference "#PWR?")
+					(unit 1)
+				)
