File: stm32_conversion_misc.kicad_sch (KiCad schematic)
At the start: 52 parts, among them IC12 LD29150DT33R, J1 MSD-4-A, U6 TXB0108PW, U7 TXB0108PW, U8 W25Q16JVSS, Y2 Crystal_GND24, Y3 Crystal_GND24

Commit message: Replace level shifters, rewire for spacing
Parts:
- removed C5, C6: 100nF, Capacitor_SMD:C_0805_2012Metric, symbol Device:C
- removed U6, U7: TXB0108PW, Package_SO:TSSOP-20_4.4x6.5mm_P0.65mm, symbol Logic_LevelTranslator:TXB0108PW
- added IC1: SN74LVC4245ADBRE4, Misc:SOP65P780X200-24N, symbol Misc:SN74LVC4245ADBRE4
- added IC13, IC14: SN74AHCT245DBR, Misc:SOP65P780X200-20N, symbol Misc:SN74AHCT245DBR
- R3: value 1k -> 10k
Connections:
- net +5V: now also IC13.20 (VCC), IC14.20 (VCC)
- net BOOST-TRIG: now also IC13.13 (B6)
- net FAN-TRIG: now also IC14.17 (B2)
- net FUELPUMP-TRIG: now also IC14.16 (B3)
- net GND: now also IC13.10 (GND), IC13.19 (~{OE}), IC14.10 (GND), IC14.19 (~{OE})
- net HC1-TRIG: now also IC13.12 (B7)
- net HC2-TRIG: now also IC13.11 (B8)
- net IDLE-TRIG: now also IC13.14 (B5)
- net IGN-1-TRIG: now also IC14.14 (B5)
- net IGN-2-TRIG: now also IC14.13 (B6)
- net IGN-3-TRIG: now also IC14.12 (B7)
- net IGN-4-TRIG: now also IC14.11 (B8)
- net INJ-1-TRIG: now also IC13.18 (B1)
- net INJ-2-TRIG: now also IC13.17 (B2)
- net INJ-3-TRIG: now also IC13.16 (B3)
- net INJ-4-TRIG: now also IC13.15 (B4)
- net LC-TRIG: now also IC14.18 (B1)
- net MCU-BOOST-TRIG-D: now also IC13.7 (A6)
- net MCU-FAN-TRIG-D: now also IC14.3 (A2)
- net MCU-FUELPUMP-TRIG-D: now also IC14.4 (A3)
- net MCU-HC-1-TRIG-D: now also IC13.8 (A7)
- net MCU-HC-2-TRIG-D: now also IC13.9 (A8)
- net MCU-IDLE-TRIG-D: now also IC13.6 (A5)
- net MCU-IGN-1-TRIG-D: now also IC14.6 (A5)
- net MCU-IGN-2-TRIG-D: now also IC14.7 (A6)
- net MCU-IGN-3-TRIG-D: now also IC14.8 (A7)
- net MCU-IGN-4-TRIG-D: now also IC14.9 (A8)
- net MCU-INJ-1-TRIG-D: now also IC13.2 (A1)
- net MCU-INJ-2-TRIG-D: now also IC13.3 (A2)
- net MCU-INJ-3-TRIG-D: now also IC13.4 (A3)
- net MCU-INJ-4-TRIG-D: now also IC13.5 (A4)
- net MCU-LC-TRIG-D: now also IC14.2 (A1)
- net MCU-TACHO-TRIG-D: now also IC14.5 (A4)
- net TACHO-TRIG: now also IC14.15 (B4)
- net at R4.2: now also IC14.1 (DIR)
- net at R3.2: now also IC13.1 (DIR)
